File: CS_Final_Project/Circuitry/Car_PCB.brd (EAGLE design)
At the start: 45.6 x 33.2 mm, 28 parts, among them SW1 KMR2, SW2 KMR2, U1 SPX3819, U2 DRV8830, X1 ESP-12, X2 22-23-2021, X3 22-23-2021

Commit message: m
Parts:
- added U$1: TCA9548A, si70xx-10:QFN24-4X4
- moved J3 32.0 mm to (15.1, 0.51), turned to 180 degrees
- moved J2 20.6 mm to (26.0, 0.51), turned to 180 degrees
- moved J1 19.2 mm to (22.2, 4.70), turned to 180 degrees
- moved JP2 12.5 mm to (34.0, 0.00), turned to 180 degrees
- moved ENCODER 8.90 mm to (6.99, 11.6), turned to 90 degrees
Connections:
- new net SC0: J1.3, U$1.5
- new net SC1: J2.3, U$1.7
- new net SC2: U$1.9
- new net SC3: J3.3, U$1.11
- new net SD0: J1.2, U$1.4
- new net SD1: J2.2, U$1.6
- new net SD2: U$1.8
- new net SD3: J3.2, U$1.10
- net 3.3V: now also J1.4, J2.4, U$1.24, U$1.3
- net GND: now also U$1.1, U$1.12, U$1.2, U$1.21
- net GPIO15: no longer J2.4
- net GPIO2: no longer J1.4
- net SCL: now also U$1.22; no longer J1.3, J2.3, J3.3
- net SDA: now also U$1.23; no longer J1.2, J2.2, J3.2
Routing:
- net 3.3V: track 95.1 -> 144.6 mm, vias 3 -> 6
- net VBAT: track 88.6 -> 133.5 mm, vias 0 -> 1
- net GPIO15: track 29.5 -> 3.60 mm, vias 1 -> 0
- net GND: track 147.4 -> 168.8 mm, vias 4 -> 5
- net GPIO2: track 24.4 -> 4.19 mm, vias 1 -> 0
- net SD1: track 0.00 -> 13.4 mm
- net SC1: track 0.00 -> 11.2 mm
- net GPIO14: track 18.0 -> 28.8 mm
- net SD0: track 0.00 -> 9.11 mm
- net GPIO12: track 12.7 -> 5.47 mm
- net SC0: track 0.00 -> 6.67 mm
- net SDA: track 53.3 -> 58.5 mm, vias 4 -> 2
- net GPIO13: track 11.5 -> 6.74 mm
- net SD3: track 0.00 -> 4.70 mm
- net SCL: track 52.4 -> 48.0 mm, vias 0 -> 2
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Other:
- board size 45.6 x 33.2 mm -> 43 x 34.7 mm
- board text added: "PWR, SCL, SDA, GND"
- board text added: "SERVO"

Commit message: m
Parts:
- removed R7: 10K, microbuilder:0805-NO
- removed U$13: (no value), microbuilder:PCBFEAT-REV-040
- added U$16: TRIN, OptoTher:TRIN
- R6: value 10K -> 10k; device microbuilder:0805-NO -> adafruit:M0805
- moved R6 29.0 mm to (3.28, 1.02), turned to 90 degrees
- moved U$1 0.18 mm to (9.40, 5.33), turned to 0 degrees
Connections:
- removed net GPIO15: R6.2, X1.10
- removed net GPIO2: R7.1, X1.11
- new net N$5: R6.2, U$1.24
- new net SC4: U$1.11
- new net SC5: J2.2, U$1.13
- new net SC6: J1.2, U$1.15
- new net SC7: U$1.17
- new net SD4: U$1.10
- new net SD5: J2.3, U$1.12
- new net SD6: J1.3, U$1.14
- new net SD7: U$1.16
- net 3.3V: now also R6.1, U$1.21, X1.11; no longer R7.2, U$1.24, U$1.3
- net GND: now also U$1.18, U$1.22, U$1.23, U$1.9, X1.10; no longer R6.1, U$1.1, U$1.12, U$1.2, U$1.21
- net SC0: now also U$1.2; no longer J1.3, U$1.5
- net SC1: now also U$1.4; no longer J2.3, U$1.7
- net SC2: now also U$1.6; no longer U$1.9
- net SC3: now also J3.2, U$1.8; no longer J3.3, U$1.11
- net SCL: now also U$1.19; no longer U$1.22
- net SD0: now also U$1.1; no longer J1.2, U$1.4
- net SD1: now also U$1.3; no longer J2.2, U$1.6
- net SD2: now also U$1.5; no longer U$1.8
- net SD3: now also J3.3, U$1.7; no longer J3.2, U$1.10
- net SDA: now also U$1.20; no longer U$1.23
Routing:
- net SC5: track 0.00 -> 13.6 mm
- net SD1: track 13.4 -> 0.00 mm
- net SD5: track 0.00 -> 11.5 mm
- net SC1: track 11.2 -> 0.00 mm
- net SC6: track 0.00 -> 9.18 mm
- net SD0: track 9.11 -> 0.00 mm
- net N$5: track 0.00 -> 9.02 mm
- net SD6: track 0.00 -> 6.75 mm
- net SC0: track 6.67 -> 0.00 mm
- net GND: track 168.8 -> 175.2 mm
- net GPIO2: track 4.19 -> 0.00 mm
- net 3.3V: track 144.6 -> 148.4 mm
- net GPIO13: track 6.74 -> 10.4 mm
- net GPIO15: track 3.60 -> 0.00 mm
- net VBAT: track 133.5 -> 130.2 mm
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Other:
- board text added: "G"
- board text added: "PWR, SDA, SCL, GND"
- board text added: "The CARS Project 2018 Charles Cunningham and Sadi Gulcelik"
- board text removed: "3.3V"
- board text removed: "CarNet Charles Cunningham and Sadi Gulcelik 2018"
- board text removed: "Contains FCC ID 2ADUIESP-12"
- board text removed: "ESP8266 WiFi 3.3V Logic Level To Bootload: hold down GPIO0 during reset"
- board text removed: "GPIO0"
- board text removed: "PWR, SCL, SDA, GND"
- board text removed: "SCL"
- board text removed: "SDA"
- board text removed: "V+: 3.5-16VDC VBat: 3.5-16VDC RX,RST: 5V OK"

Commit message: Revert "Merge branch 'master' of https://github.com/mureytasroc/CarNetwork"
This reverts commit a45a0045a92c6dc43e66f74dc99afbd22e46fa88, reversing
changes made to 7d7a9c1b56f2fe83920f8a54f55361a334df6815.
Parts:
- removed U$16: TRIN, OptoTher:TRIN
- added R7: 10K, microbuilder:0805-NO
- added U$13: (no value), microbuilder:PCBFEAT-REV-040
- R6: value 10k -> 10K; device adafruit:M0805 -> microbuilder:0805-NO
- moved R6 29.0 mm to (30.9, 10.0), turned to 180 degrees
- moved U$1 0.18 mm to (9.53, 5.21), turned to 270 degrees
Connections:
- removed net N$5: R6.2, U$1.24
- removed net SC4: U$1.11
- removed net SC5: J2.2, U$1.13
- removed net SC6: J1.2, U$1.15
- removed net SC7: U$1.17
- removed net SD4: U$1.10
- removed net SD5: J2.3, U$1.12
- removed net SD6: J1.3, U$1.14
- removed net SD7: U$1.16
- new net GPIO15: R6.2, X1.10
- new net GPIO2: R7.1, X1.11
- net 3.3V: now also R7.2, U$1.24, U$1.3; no longer R6.1, U$1.21, X1.11
- net GND: now also R6.1, U$1.1, U$1.12, U$1.2, U$1.21; no longer U$1.18, U$1.22, U$1.23, U$1.9, X1.10
- net SC0: now also J1.3, U$1.5; no longer U$1.2
- net SC1: now also J2.3, U$1.7; no longer U$1.4
- net SC2: now also U$1.9; no longer U$1.6
- net SC3: now also J3.3, U$1.11; no longer J3.2, U$1.8
- net SCL: now also U$1.22; no longer U$1.19
- net SD0: now also J1.2, U$1.4; no longer U$1.1
- net SD1: now also J2.2, U$1.6; no longer U$1.3
- net SD2: now also U$1.8; no longer U$1.5
- net SD3: now also J3.2, U$1.10; no longer J3.3, U$1.7
- net SDA: now also U$1.23; no longer U$1.20
Routing:
- net SC5: track 13.6 -> 0.00 mm
- net SD1: track 0.00 -> 13.4 mm
- net SD5: track 11.5 -> 0.00 mm
- net SC1: track 0.00 -> 11.2 mm
- net SC6: track 9.18 -> 0.00 mm
- net SD0: track 0.00 -> 9.11 mm
- net N$5: track 9.02 -> 0.00 mm
- net SD6: track 6.75 -> 0.00 mm
- net SC0: track 0.00 -> 6.67 mm
- net GND: track 175.2 -> 168.8 mm
- net GPIO2: track 0.00 -> 4.19 mm
- net 3.3V: track 148.4 -> 144.6 mm
- net GPIO13: track 10.4 -> 6.74 mm
- net GPIO15: track 0.00 -> 3.60 mm
- net VBAT: track 130.2 -> 133.5 mm
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Other:
- board text added: "3.3V"
- board text added: "CarNet Charles Cunningham and Sadi Gulcelik 2018"
- board text added: "Contains FCC ID 2ADUIESP-12"
- board text added: "ESP8266 WiFi 3.3V Logic Level To Bootload: hold down GPIO0 during reset"
- board text added: "GPIO0"
- board text added: "PWR, SCL, SDA, GND"
- board text added: "SCL"
- board text added: "SDA"
- board text added: "V+: 3.5-16VDC VBat: 3.5-16VDC RX,RST: 5V OK"
- board text removed: "G"
- board text removed: "PWR, SDA, SCL, GND"
- board text removed: "The CARS Project 2018 Charles Cunningham and Sadi Gulcelik"
