File: CS_Final_Project/Circuitry/Car_PCB.sch (EAGLE design)
At the start: 25 parts, among them SW1 KMR2, SW2 KMR2, U1 SPX3819, U2 DRV8830, X1 ESP-12, X2 22-23-2021, X3 22-23-2021

Commit message: m
Other:
- note added: "Dont connect GPIO2 and pull down gpio15 with 1k in future versions"
Changed lines of the file:
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@@
 <text x="121.92" y="50.8" size="1.778" layer="97">B GPIO13</text>
 <text x="68.58" y="43.18" size="1.778" layer="97">3.3</text>
+<text x="121.92" y="111.76" size="1.778" layer="97">Dont connect GPIO2 and pull down gpio15 with 1k in future versions</text>
 </plain>
 <instances>
